Commit message: Full update Omni Wheel Mobile

File: lib_omni_mobile/urdf/omni_mobile.xacro (robot description, xacro)
@@ -2,10 +2,9 @@
 <robot xmlns:xacro="http://www.ros.org/wiki/xacro" name="omni_mobile">
     <xacro:include filename="$(find lib_omni_mobile)/urdf/materials.xacro" />
-	<xacro:property name="offset" value="0.02" />
 	<xacro:property name="PI" value="3.14" />
     <xacro:property name="base_link_length" value="0.1" />
     <xacro:property name="base_link_radius" value="0.2" />
 	<xacro:property name="wheel_length" value="0.05" />
-	<xacro:property name="wheel_radius" value="0.02" />
+	<xacro:property name="wheel_radius" value="0.1" />
     <link name="base_link">
 		<visual>
@@ -13,5 +12,5 @@
 				<cylinder length="${base_link_length}" radius="${base_link_radius}"/>
 			</geometry>
-			<origin xyz="0.0 0.0 ${base_link_length/2 + wheel_radius/2}"/>
+			<origin xyz="0 0 ${base_link_length/2+wheel_radius/2}"/>
 			<material name="blue"/>
 		</visual>
@@ -20,5 +19,5 @@
 				<cylinder length="${base_link_length}" radius="${base_link_radius}"/>
 			</geometry>
-			<origin xyz="0.0 0.0 ${base_link_length/2 + wheel_radius/2}"/>
+			<origin xyz="0 0 ${base_link_length/2+wheel_radius/2}"/>
 			<material name="blue"/>
 		</collision>
@@ -27,6 +26,6 @@
 		<parent link="base_link"/>
 		<child link="wheel_1"/>
-		<origin xyz="0.0 0.0 ${base_link_length+offset}"/>
-		<axis xyz="0 1 0"/>
+		<origin xyz="${base_link_radius+wheel_length/2} 0 ${base_link_length}" rpy="0 ${PI/2} 0"/>
+		<axis xyz="0 0 1"/>
 		<limit effort="1000" lower="${-PI}" upper="${PI}" velocity="5"/>
 	</joint>
@@ -36,5 +35,5 @@
 				<cylinder length="${wheel_length}" radius="${wheel_radius}"/>
 			</geometry>
-			<origin xyz="0.0 0.0 ${wheel_length/2}"/>
+			<origin xyz="0 0 0"/>
 			<material name="black"/>
 		</visual>
@@ -43,5 +42,51 @@
 				<cylinder length="${wheel_length}" radius="${wheel_radius}"/>
 			</geometry>
-			<origin xyz="0.0 0.0 ${wheel_length/2}"/>
+			<origin xyz="0 0 0"/>
+			<material name="black"/>
+		</collision>
+	</link>
+	<joint name="jwheel_2" type="revolute">
+		<parent link="base_link"/>
+		<child link="wheel_2"/>
+		<origin xyz="${-0.5*(base_link_radius+wheel_length/2)} ${0.866*(base_link_radius+wheel_length/2)} ${base_link_length}" rpy="0 ${PI/2} ${2*PI/3}"/>
+		<axis xyz="0 0 1"/>
+		<limit effort="1000" lower="${-PI}" upper="${PI}" velocity="5"/>
+	</joint>
+	<link name="wheel_2">
+		<visual>
+			<geometry>
+				<cylinder length="${wheel_length}" radius="${wheel_radius}"/>
+			</geometry>
+			<origin xyz="0 0 0"/>
+			<material name="black"/>
+		</visual>
+		<collision>
+			<geometry>
+				<cylinder length="${wheel_length}" radius="${wheel_radius}"/>
+			</geometry>
+			<origin xyz="0 0 0"/>
+			<material name="black"/>
+		</collision>
+	</link>
+	<joint name="jwheel_3" type="revolute">
+		<parent link="base_link"/>
+		<child link="wheel_3"/>
+		<origin xyz="${-0.5*(base_link_radius+wheel_length/2)} ${-0.866*(base_link_radius+wheel_length/2)} ${base_link_length}" rpy="0 ${PI/2} ${-2*PI/3}"/>
+		<axis xyz="0 0 1"/>
+		<limit effort="1000" lower="${-PI}" upper="${PI}" velocity="5"/>
+	</joint>
+	<link name="wheel_3">
+		<visual>
+			<geometry>
+				<cylinder length="${wheel_length}" radius="${wheel_radius}"/>
+			</geometry>
+			<origin xyz="0 0 0"/>
+			<material name="black"/>
+		</visual>
+		<collision>
+			<geometry>
+				<cylinder length="${wheel_length}" radius="${wheel_radius}"/>
+			</geometry>
+			<origin xyz="0 0 0"/>
 			<material name="black"/>
 		</collision>

Commit message: Update code Omni

File: lib_omni_mobile/urdf/omni_mobile.xacro (robot description, xacro)
@@ -4,6 +4,6 @@
 	<xacro:property name="PI" value="3.14" />
     <xacro:property name="base_link_length" value="0.1" />
-    <xacro:property name="base_link_radius" value="0.2" />
-	<xacro:property name="wheel_length" value="0.05" />
+    <xacro:property name="base_link_radius" value="0.15" />
+	<xacro:property name="wheel_length" value="0.035" />
 	<xacro:property name="wheel_radius" value="0.1" />
     <link name="base_link">
