Commit message: Add SLAM

File: lib_omni_mobile/urdf/omni_mobile.urdf.xacro (robot description, xacro)
@@ -2,4 +2,5 @@
 <robot xmlns:xacro="http://www.ros.org/wiki/xacro" name="omni_mobile">
     <xacro:include filename="$(find lib_omni_mobile)/urdf/materials.xacro" />
+	<xacro:include filename="$(find lib_omni_mobile)/urdf/roller_wheel.urdf.xacro"/>
 	<xacro:include filename="$(find lib_omni_mobile)/urdf/omni_mobile.gazebo.xacro" />
 	<xacro:property name="PI" value="3.14" />
@@ -27,11 +28,4 @@
 			<material name="blue"/>
 		</collision>
-		<!-- <inertial>
-			<origin xyz="0.0 0 0.0" rpy="0 0 0"/>
-			<mass value="1.6329594e+00"/>
-			<inertia ixx="1.0" ixy="0.0" ixz="0.0"
-					iyy="1.0" iyz="0.0"
-					izz="1.0" />
-		</inertial> -->
 	</link>
 	<joint name="jwheel_1" type="continuous">
@@ -134,5 +128,4 @@
 			<origin xyz="0 0 0"/>
 			<geometry>
-				<!-- <cylinder length="0.0315" radius="0.045"/> -->
 				<mesh filename="package://turtlebot3_description/meshes/sensors/lds.stl" scale="0.001 0.001 0.001"/>
 			</geometry>
@@ -155,9 +148,3 @@
 		</inertial>
 	</link>
-	<!-- <joint name="imu_joint" type="fixed">
-    	<parent link="base_link"/>
-    	<child link="imu_link"/>
-    	<origin xyz="0.0 0 0.068" rpy="0 0 0"/>
-  	</joint>
-  	<link name="imu_link"/> -->
 </robot>

Commit message: Mini Update

File: lib_omni_mobile/urdf/omni_mobile.urdf.xacro (robot description, xacro)
@@ -29,7 +29,7 @@
 		</inertial>
 	</link>
-	<xacro:rim name="left_wheel" parent="base_link" xyz="${-0.5*(base_link_radius+wheel_length/2)} ${0.866*(base_link_radius+wheel_length/2)} ${base_link_length}" rpy="0 ${PI/2} ${2*PI/3}"/>
-	<xacro:rim name="right_wheel" parent="base_link" xyz="${-0.5*(base_link_radius+wheel_length/2)} ${-0.866*(base_link_radius+wheel_length/2)} ${base_link_length}" rpy="0 ${PI/2} ${-2*PI/3}"/>
-	<xacro:rim name="front_wheel" parent="base_link" xyz="${base_link_radius+wheel_length/2} 0 ${base_link_length}" rpy="0 ${PI/2} ${PI}"/>
+	<xacro:rim name="left_wheel" parent="base_link" xyz="${-0.5*(base_link_radius+wheel_length/2)} ${0.866*(base_link_radius+wheel_length/2)} ${-base_link_length}" rpy="0 ${PI/2} ${2*PI/3}"/>
+	<xacro:rim name="right_wheel" parent="base_link" xyz="${-0.5*(base_link_radius+wheel_length/2)} ${-0.866*(base_link_radius+wheel_length/2)} ${-base_link_length}" rpy="0 ${PI/2} ${-2*PI/3}"/>
+	<xacro:rim name="front_wheel" parent="base_link" xyz="${base_link_radius+wheel_length/2} 0 ${-base_link_length}" rpy="0 ${PI/2} ${PI}"/>
 	<joint name="scan_joint" type="fixed">
 		<parent link="base_link"/>
@@ -44,5 +44,5 @@
 			</geometry>
 			<origin xyz="0 0 0" rpy="0 0 0"/>
-			<material name="dark"/>
+			<material name="black"/>
 		</visual>
 	</link>

Commit message: Add new Nav

File: lib_omni_mobile/urdf/omni_mobile.urdf.xacro (robot description, xacro)
@@ -4,8 +4,10 @@
 	<xacro:include filename="$(find lib_omni_mobile)/urdf/omni_mobile.gazebo.xacro" />
 	<xacro:property name="PI" value="3.14" />
-    <xacro:property name="base_link_length" value="0.07" />
+    <xacro:property name="base_link_length" value="0.12" />
     <xacro:property name="base_link_radius" value="0.15" />
-	<xacro:property name="wheel_length" value="0.04" />
-	<xacro:property name="wheel_radius" value="0.04" />
+	<xacro:property name="wheel_length" value="0.036" />
+	<xacro:property name="wheel_radius" value="0.032" />
+	<xacro:property name="roller_length" value="0.018" />
+	<xacro:property name="roller_radius" value="0.009" />
     <link name="base_link">
 		<visual>
@@ -13,5 +15,5 @@
 				<cylinder length="${base_link_length}" radius="${base_link_radius}"/>
 			</geometry>
-			<origin xyz="0 0 ${base_link_length/2+wheel_radius}" rpy="0 0 0"/>
+			<origin xyz="0 0 ${base_link_length/2+roller_length}" rpy="0 0 0"/>
 			<material name="white"/>
 		</visual>
@@ -20,5 +22,5 @@
 				<cylinder length="${base_link_length}" radius="${base_link_radius}"/>
 			</geometry>
-			<origin xyz="0 0 ${base_link_length/2+wheel_radius}" rpy="0 0 0"/>
+			<origin xyz="0 0 ${base_link_length/2+roller_length}" rpy="0 0 0"/>
 			<material name="white"/>
 		</collision>
@@ -29,11 +31,11 @@
 		</inertial>
 	</link>
-	<xacro:rim name="left_wheel" parent="base_link" xyz="${-0.5*(base_link_radius+wheel_length/2)} ${0.866*(base_link_radius+wheel_length/2)} ${-base_link_length}" rpy="0 ${PI/2} ${2*PI/3}"/>
-	<xacro:rim name="right_wheel" parent="base_link" xyz="${-0.5*(base_link_radius+wheel_length/2)} ${-0.866*(base_link_radius+wheel_length/2)} ${-base_link_length}" rpy="0 ${PI/2} ${-2*PI/3}"/>
-	<xacro:rim name="front_wheel" parent="base_link" xyz="${base_link_radius+wheel_length/2} 0 ${-base_link_length}" rpy="0 ${PI/2} ${PI}"/>
+	<xacro:rim name="left_wheel" parent="base_link" xyz="${0.5*(base_link_radius+wheel_length/2)} ${0.866*(base_link_radius+wheel_length/2)} ${base_link_length/2-roller_radius}" rpy="0 ${PI/2} ${PI/3}"/>
+	<xacro:rim name="right_wheel" parent="base_link" xyz="${0.5*(base_link_radius+wheel_length/2)} ${-0.866*(base_link_radius+wheel_length/2)} ${base_link_length/2-roller_radius}" rpy="0 ${PI/2} ${-PI/3}"/>
+	<xacro:rim name="front_wheel" parent="base_link" xyz="${-base_link_radius-wheel_length/2} 0 ${base_link_length/2-roller_radius}" rpy="0 ${PI/2} ${PI}"/>
 	<joint name="scan_joint" type="fixed">
 		<parent link="base_link"/>
 		<child link="base_scan"/>
-		<origin xyz="-0.024 0 0.17" rpy="0 0 0"/>
+		<origin xyz="${base_link_radius-wheel_length/2} 0 ${base_link_length+roller_radius*4}" rpy="0 0 0"/>
   	</joint>
 	<link name="base_scan">

File: lib_omni_mobile/urdf/rim_wheel.urdf.xacro (robot description, xacro)
@@ -10,5 +10,5 @@
         <visual>
             <geometry>
-                <cylinder radius="0.04" length="0.04"/>
+                <cylinder radius="0.032" length="0.036"/>
             </geometry>
             <material name="black"/>
@@ -16,5 +16,5 @@
         <collision>
             <geometry>
-                <cylinder radius="0.04" length="0.04"/>
+                <cylinder radius="0.032" length="0.036"/>
             </geometry>
             <material name="black"/>
@@ -28,20 +28,20 @@
         <limit effort="1000" velocity="3140"/>
     </joint>
-    <xacro:roller name="8" parent="${name}"  xyz="0.05 0 0.01" rpy="1.57 0 0"/>
-	<xacro:roller name="7" parent="${name}"  xyz="0.046194 0.019134 -0.01" rpy="1.57 0 0.3927"/>
-	<xacro:roller name="6" parent="${name}"  xyz="0.035355 0.035355 0.01" rpy="1.57 0 0.7854"/>
-	<xacro:roller name="5" parent="${name}"  xyz="0.019134 0.046194 -0.01" rpy="1.57 0 1.1781"/>
-	<xacro:roller name="4" parent="${name}"  xyz="0 0.05 0.01" rpy="1.57 0 1.5708"/>
-	<xacro:roller name="3" parent="${name}"  xyz="-0.019134 0.046194 -0.01" rpy="1.57 0 1.9635"/>
-	<xacro:roller name="2" parent="${name}"  xyz="-0.035355 0.035355 0.01" rpy="1.57 0 2.3562"/>
-	<xacro:roller name="1" parent="${name}"  xyz="-0.046194 0.019134 -0.01" rpy="1.57 0 2.7489"/>
-	<xacro:roller name="16" parent="${name}" xyz="-0.05 0 0.01" rpy="1.57 0 3.1416"/>
-	<xacro:roller name="15" parent="${name}" xyz="-0.046194 -0.019134 -0.01" rpy="1.57 0 -2.7489"/>
-	<xacro:roller name="14" parent="${name}" xyz="-0.035355 -0.035355 0.01" rpy="1.57 0 -2.3562"/>
-	<xacro:roller name="13" parent="${name}" xyz="-0.019134 -0.046194 -0.01" rpy="1.57 0 -1.9635"/>
-	<xacro:roller name="12" parent="${name}" xyz="0 -0.05 0.01" rpy="1.57 0 -1.5708"/>
-	<xacro:roller name="11" parent="${name}" xyz="0.019134 -0.046194 -0.01" rpy="1.57 0 -1.1781"/>
-	<xacro:roller name="10" parent="${name}" xyz="0.035355 -0.035355 0.01" rpy="1.57 0 -0.7854"/>
-	<xacro:roller name="9" parent="${name}" xyz="0.046194 -0.019134 -0.01" rpy="1.57 0 -0.3927"/>
+    <xacro:roller name="8" parent="${name}"  xyz="0.041 0 0.01" rpy="1.57 0 0"/>
+	<xacro:roller name="7" parent="${name}"  xyz="0.037879 0.015690 -0.01" rpy="1.57 0 0.3927"/>
+	<xacro:roller name="6" parent="${name}"  xyz="0.028991 0.028991 0.01" rpy="1.57 0 0.7854"/>
+	<xacro:roller name="5" parent="${name}"  xyz="0.015690 0.037879 -0.01" rpy="1.57 0 1.1781"/>
+	<xacro:roller name="4" parent="${name}"  xyz="0 0.041 0.01" rpy="1.57 0 1.5708"/>
+	<xacro:roller name="3" parent="${name}"  xyz="-0.015690 0.037879 -0.01" rpy="1.57 0 1.9635"/>
+	<xacro:roller name="2" parent="${name}"  xyz="-0.028991 0.028991 0.01" rpy="1.57 0 2.3562"/>
+	<xacro:roller name="1" parent="${name}"  xyz="-0.037879 0.015690 -0.01" rpy="1.57 0 2.7489"/>
+	<xacro:roller name="16" parent="${name}" xyz="-0.041 0 0.01" rpy="1.57 0 3.1416"/>
+	<xacro:roller name="15" parent="${name}" xyz="-0.037879 -0.015690 -0.01" rpy="1.57 0 -2.7489"/>
+	<xacro:roller name="14" parent="${name}" xyz="-0.028991 -0.028991 0.01" rpy="1.57 0 -2.3562"/>
+	<xacro:roller name="13" parent="${name}" xyz="-0.015690 -0.037879 -0.01" rpy="1.57 0 -1.9635"/>
+	<xacro:roller name="12" parent="${name}" xyz="0 -0.041 0.01" rpy="1.57 0 -1.5708"/>
+	<xacro:roller name="11" parent="${name}" xyz="0.015690 -0.037879 -0.01" rpy="1.57 0 -1.1781"/>
+	<xacro:roller name="10" parent="${name}" xyz="0.028991 -0.028991 0.01" rpy="1.57 0 -0.7854"/>
+	<xacro:roller name="9" parent="${name}" xyz="0.037879 -0.015690 -0.01" rpy="1.57 0 -0.3927"/>
     <transmission name="${name}_tran">
         <type>transmission_interface/SimpleTransmission</type>

File: lib_omni_mobile/urdf/roller_wheel.urdf.xacro (robot description, xacro)
@@ -9,10 +9,10 @@
         <visual>
             <geometry>
-                <cylinder radius="0.01" length="0.02"/>
+                <cylinder radius="0.009" length="0.018"/>
             </geometry>
         </visual>
         <collision>
             <geometry>
-                <cylinder radius="0.01" length="0.02"/>
+                <cylinder radius="0.009" length="0.018"/>
             </geometry>
         </collision>
