Commit message: Big Update Before Demo

File: lib_omni_mobile/urdf/omni_mobile.gazebo.xacro (robot description, xacro)
@@ -7,6 +7,6 @@
     <material>Gazebo/DarkGrey</material>
   </gazebo>
-  <!-- <gazebo reference="front_wheel">
-    <mu1>10000</mu1>
+  <gazebo reference="front_wheel">
+    <!-- <mu1>10000</mu1>
     <mu2>10000</mu2>
     <kp>500000.0</kp>
@@ -14,9 +14,9 @@
     <minDepth>0.001</minDepth>
     <maxVel>0.1</maxVel>
-    <fdir1>1 0 0</fdir1>
+    <fdir1>1 0 0</fdir1> -->
     <material>Gazebo/FlatBlack</material>
-  </gazebo> -->
-  <!-- <gazebo reference="left_wheel">
-    <mu1>10000</mu1>
+  </gazebo>
+  <gazebo reference="left_wheel">
+    <!-- <mu1>10000</mu1>
     <mu2>10000</mu2>
     <kp>500000.0</kp>
@@ -24,9 +24,9 @@
     <minDepth>0.001</minDepth>
     <maxVel>0.1</maxVel>
-    <fdir1>1 0 0</fdir1>
+    <fdir1>1 0 0</fdir1> -->
     <material>Gazebo/FlatBlack</material>
-  </gazebo> -->
-  <!-- <gazebo reference="right_wheel">
-    <mu1>10000</mu1>
+  </gazebo>
+  <gazebo reference="right_wheel">
+    <!-- <mu1>10000</mu1>
     <mu2>10000</mu2>
     <kp>500000.0</kp>
@@ -34,7 +34,7 @@
     <minDepth>0.001</minDepth>
     <maxVel>0.1</maxVel>
-    <fdir1>1 0 0</fdir1>
+    <fdir1>1 0 0</fdir1> -->
     <material>Gazebo/FlatBlack</material>
-  </gazebo> -->
+  </gazebo>
   <!-- <gazebo reference="imu_link">
     <sensor type="imu" name="imu">
@@ -59,5 +59,5 @@
     </plugin>
   </gazebo> -->
-  <!-- <gazebo reference="imu_link">
+  <gazebo reference="imu_link">
     <gravity>true</gravity>
     <sensor name="imu_sensor" type="imu">
@@ -67,5 +67,5 @@
       <topic>__default_topic__</topic>
       <plugin filename="libgazebo_ros_imu_sensor.so" name="imu_plugin">
-        <topicName>imu_data</topicName>
+        <topicName>imu</topicName>
         <bodyName>imu_link</bodyName>
         <updateRateHZ>10.0</updateRateHZ>
@@ -78,5 +78,5 @@
       <pose>0 0 0 0 0 0</pose>
     </sensor>
-  </gazebo> -->
+  </gazebo>
   <!-- <gazebo>
     <plugin name="imu_plugin" filename="libgazebo_ros_imu.so">

File: lib_omni_mobile/urdf/omni_mobile.urdf.xacro (robot description, xacro)
@@ -4,10 +4,10 @@
 	<xacro:include filename="$(find lib_omni_mobile)/urdf/omni_mobile.gazebo.xacro" />
 	<xacro:property name="PI" value="3.14" />
-    <xacro:property name="base_link_length" value="0.12" />
-    <xacro:property name="base_link_radius" value="0.15" />
-	<xacro:property name="wheel_length" value="0.036" />
-	<xacro:property name="wheel_radius" value="0.032" />
-	<xacro:property name="roller_length" value="0.018" />
-	<xacro:property name="roller_radius" value="0.009" />
+    <xacro:property name="base_link_length" value="0.124" />
+    <xacro:property name="base_link_radius" value="0.14256" />
+	<xacro:property name="wheel_length" value="0.029" />
+	<xacro:property name="wheel_radius" value="0.0435" />
+	<xacro:property name="roller_length" value="0.0186" />
+	<xacro:property name="roller_radius" value="0.0095" />
     <link name="base_link">
 		<visual>
@@ -15,5 +15,5 @@
 				<cylinder length="${base_link_length}" radius="${base_link_radius}"/>
 			</geometry>
-			<origin xyz="0 0 ${base_link_length/2+roller_length}" rpy="0 0 0"/>
+			<origin xyz="0 0 0" rpy="0 0 0"/>
 			<material name="white"/>
 		</visual>
@@ -22,5 +22,5 @@
 				<cylinder length="${base_link_length}" radius="${base_link_radius}"/>
 			</geometry>
-			<origin xyz="0 0 ${base_link_length/2+roller_length}" rpy="0 0 0"/>
+			<origin xyz="0 0 0" rpy="0 0 0"/>
 			<material name="white"/>
 		</collision>
@@ -31,11 +31,11 @@
 		</inertial>
 	</link>
-	<xacro:rim name="left_wheel" parent="base_link" xyz="${0.5*(base_link_radius+wheel_length/2)} ${0.866*(base_link_radius+wheel_length/2)} ${base_link_length/2-roller_radius}" rpy="0 ${PI/2} ${PI/3}"/>
-	<xacro:rim name="right_wheel" parent="base_link" xyz="${0.5*(base_link_radius+wheel_length/2)} ${-0.866*(base_link_radius+wheel_length/2)} ${base_link_length/2-roller_radius}" rpy="0 ${PI/2} ${-PI/3}"/>
-	<xacro:rim name="front_wheel" parent="base_link" xyz="${-base_link_radius-wheel_length/2} 0 ${base_link_length/2-roller_radius}" rpy="0 ${PI/2} ${PI}"/>
+	<xacro:rim name="left_wheel" parent="base_link" xyz="${-0.5*(base_link_radius+wheel_length/2+0.017)} ${0.866*(base_link_radius+wheel_length/2+0.017)} ${-0.03235}" rpy="0 ${PI/2} ${-PI/3}"/>
+	<xacro:rim name="right_wheel" parent="base_link" xyz="${-0.5*(base_link_radius+wheel_length/2+0.017)} ${-0.866*(base_link_radius+wheel_length/2+0.017)} ${-0.03235}" rpy="0 ${PI/2} ${PI/3}"/>
+	<xacro:rim name="front_wheel" parent="base_link" xyz="${base_link_radius+wheel_length/2+0.017} 0 ${-0.03235}" rpy="0 ${PI/2} ${PI}"/>
 	<joint name="scan_joint" type="fixed">
 		<parent link="base_link"/>
 		<child link="base_scan"/>
-		<origin xyz="${base_link_radius-wheel_length/2} 0 ${base_link_length+roller_radius*4}" rpy="0 0 0"/>
+		<origin xyz="${-(base_link_radius-wheel_length/2)} 0 ${base_link_length-0.03235}" rpy="0 0 ${PI}"/>
   	</joint>
 	<link name="base_scan">
@@ -43,6 +43,5 @@
 			<origin xyz="0 0 0"/>
 			<geometry>
-				<!-- <mesh filename="package://turtlebot3_description/meshes/sensors/lds.stl" scale="0.001 0.001 0.001"/> -->
-				<cylinder length="0.05" radius="0.02"/>
+				<mesh filename="package://lib_omni_mobile/meshes/lds.stl" scale="0.001 0.001 0.001"/>
 			</geometry>
 			<origin xyz="0 0 0" rpy="0 0 0"/>
@@ -50,9 +49,9 @@
 		</visual>
 	</link>
-	<!-- <joint name="imu_joint" type="fixed">
+	<joint name="imu_joint" type="fixed">
     	<parent link="base_link"/>
     	<child link="imu_link"/>
     	<origin xyz="0.0 0.0 0.0" rpy="0 0 0"/>
   	</joint>
-  	<link name="imu_link"/> -->
+  	<link name="imu_link"/>
 </robot>

File: lib_omni_mobile/urdf/rim_wheel.urdf.xacro (robot description, xacro)
@@ -10,5 +10,5 @@
         <visual>
             <geometry>
-                <cylinder radius="0.032" length="0.036"/>
+                <cylinder radius="0.0435" length="0.029"/>
             </geometry>
             <material name="black"/>
@@ -16,5 +16,5 @@
         <collision>
             <geometry>
-                <cylinder radius="0.032" length="0.036"/>
+                <cylinder radius="0.0435" length="0.029"/>
             </geometry>
             <material name="black"/>
@@ -28,20 +28,20 @@
         <limit effort="1000" velocity="3140"/>
     </joint>
-    <xacro:roller name="8" parent="${name}"  xyz="0.041 0 0.01" rpy="1.57 0 0"/>
-	<xacro:roller name="7" parent="${name}"  xyz="0.037879 0.015690 -0.01" rpy="1.57 0 0.3927"/>
-	<xacro:roller name="6" parent="${name}"  xyz="0.028991 0.028991 0.01" rpy="1.57 0 0.7854"/>
-	<xacro:roller name="5" parent="${name}"  xyz="0.015690 0.037879 -0.01" rpy="1.57 0 1.1781"/>
-	<xacro:roller name="4" parent="${name}"  xyz="0 0.041 0.01" rpy="1.57 0 1.5708"/>
-	<xacro:roller name="3" parent="${name}"  xyz="-0.015690 0.037879 -0.01" rpy="1.57 0 1.9635"/>
-	<xacro:roller name="2" parent="${name}"  xyz="-0.028991 0.028991 0.01" rpy="1.57 0 2.3562"/>
-	<xacro:roller name="1" parent="${name}"  xyz="-0.037879 0.015690 -0.01" rpy="1.57 0 2.7489"/>
-	<xacro:roller name="16" parent="${name}" xyz="-0.041 0 0.01" rpy="1.57 0 3.1416"/>
-	<xacro:roller name="15" parent="${name}" xyz="-0.037879 -0.015690 -0.01" rpy="1.57 0 -2.7489"/>
-	<xacro:roller name="14" parent="${name}" xyz="-0.028991 -0.028991 0.01" rpy="1.57 0 -2.3562"/>
-	<xacro:roller name="13" parent="${name}" xyz="-0.015690 -0.037879 -0.01" rpy="1.57 0 -1.9635"/>
-	<xacro:roller name="12" parent="${name}" xyz="0 -0.041 0.01" rpy="1.57 0 -1.5708"/>
-	<xacro:roller name="11" parent="${name}" xyz="0.015690 -0.037879 -0.01" rpy="1.57 0 -1.1781"/>
-	<xacro:roller name="10" parent="${name}" xyz="0.028991 -0.028991 0.01" rpy="1.57 0 -0.7854"/>
-	<xacro:roller name="9" parent="${name}" xyz="0.037879 -0.015690 -0.01" rpy="1.57 0 -0.3927"/>
+    <xacro:roller name="8" parent="${name}"  xyz="0.053 0 0.0095" rpy="1.57 0 0"/>
+	<xacro:roller name="7" parent="${name}"  xyz="0.048966 0.020282 -0.0095" rpy="1.57 0 0.3927"/>
+	<xacro:roller name="6" parent="${name}"  xyz="0.037477 0.037477 0.0095" rpy="1.57 0 0.7854"/>
+	<xacro:roller name="5" parent="${name}"  xyz="0.020282 0.048966 -0.0095" rpy="1.57 0 1.1781"/>
+	<xacro:roller name="4" parent="${name}"  xyz="0 0.053 0.0095" rpy="1.57 0 1.5708"/>
+	<xacro:roller name="3" parent="${name}"  xyz="-0.020282 0.048966 -0.0095" rpy="1.57 0 1.9635"/>
+	<xacro:roller name="2" parent="${name}"  xyz="-0.037477 0.037477 0.0095" rpy="1.57 0 2.3562"/>
+	<xacro:roller name="1" parent="${name}"  xyz="-0.048966 0.020282 -0.0095" rpy="1.57 0 2.7489"/>
+	<xacro:roller name="16" parent="${name}" xyz="-0.053 0 0.0095" rpy="1.57 0 3.1416"/>
+	<xacro:roller name="15" parent="${name}" xyz="-0.048966 -0.020282 -0.0095" rpy="1.57 0 -2.7489"/>
+	<xacro:roller name="14" parent="${name}" xyz="-0.037477 -0.037477 0.0095" rpy="1.57 0 -2.3562"/>
+	<xacro:roller name="13" parent="${name}" xyz="-0.020282 -0.048966 -0.0095" rpy="1.57 0 -1.9635"/>
+	<xacro:roller name="12" parent="${name}" xyz="0 -0.053 0.0095" rpy="1.57 0 -1.5708"/>
+	<xacro:roller name="11" parent="${name}" xyz="0.020282 -0.048966 -0.0095" rpy="1.57 0 -1.1781"/>
+	<xacro:roller name="10" parent="${name}" xyz="0.037477 -0.037477 0.0095" rpy="1.57 0 -0.7854"/>
+	<xacro:roller name="9" parent="${name}" xyz="0.048966 -0.020282 -0.0095" rpy="1.57 0 -0.3927"/>
     <transmission name="${name}_tran">
         <type>transmission_interface/SimpleTransmission</type>

File: lib_omni_mobile/urdf/roller_wheel.urdf.xacro (robot description, xacro)
@@ -9,10 +9,10 @@
         <visual>
             <geometry>
-                <cylinder radius="0.009" length="0.018"/>
+                <cylinder radius="0.0095" length="0.0186"/>
             </geometry>
         </visual>
         <collision>
             <geometry>
-                <cylinder radius="0.009" length="0.018"/>
+                <cylinder radius="0.0095" length="0.0186"/>
             </geometry>
         </collision>
