Commit message: Big Update

File: lib_bringup/urdf/librarian.urdf.xacro (robot description, xacro)
@@ -1,13 +1,14 @@
 <?xml version="1.0"?>
 <robot name="librarian" xmlns:xacro="http://ros.org/wiki/xacro">
-  <!-- Include TurtleBot3 Waffle URDF -->
-  <xacro:include filename="$(find lib_bringup)/urdf/turtlebot3_waffle_pi_for_open_manipulator.urdf.xacro"/>
-  <!-- Include OpenMANIPULATOR URDF -->
-  <xacro:include filename="$(find lib_bringup)/urdf/open_manipulator_x.urdf.xacro"/>
+  <xacro:include filename="$(find lib_bringup)/urdf/materials.xacro" />
+  <!-- Include Omni Mobile URDF -->
+  <xacro:include filename="$(find lib_omni_mobile)/urdf/omni_mobile.urdf.xacro" />
+  <!-- Include Planar Arm URDF -->
+  <xacro:include filename="$(find lib_planar_arm)/urdf/planar_arm.urdf.xacro" />
   <!-- Base fixed joint -->
   <joint name="base_fixed" type="fixed">
-    <origin xyz="-0.092 0.0 0.091" rpy="0 0 0"/>
+    <origin xyz="0.0 0.0 0.0" rpy="0 0 0"/>
     <parent link="base_link"/>
-    <child link="link1"/>
+    <child link="planar_link"/>
   </joint>
 </robot>

File: lib_omni_mobile/urdf/omni_mobile.gazebo.xacro (robot description, xacro)
@@ -1,4 +1,4 @@
 <?xml version="1.0"?>
-<robot name="omni_mobile" xmlns:xacro="http://ros.org/wiki/xacro">
+<robot xmlns:xacro="http://www.ros.org/wiki/xacro">
   <xacro:arg name="laser_visual"  default="false"/>
   <xacro:arg name="camera_visual" default="false"/>
@@ -7,5 +7,5 @@
     <material>Gazebo/DarkGrey</material>
   </gazebo>
-  <!-- <gazebo reference="wheel_1">
+  <!-- <gazebo reference="front_wheel">
     <mu1>10000</mu1>
     <mu2>10000</mu2>
@@ -17,5 +17,5 @@
     <material>Gazebo/FlatBlack</material>
   </gazebo> -->
-  <!-- <gazebo reference="wheel_2">
+  <!-- <gazebo reference="left_wheel">
     <mu1>10000</mu1>
     <mu2>10000</mu2>
@@ -27,5 +27,5 @@
     <material>Gazebo/FlatBlack</material>
   </gazebo> -->
-  <!-- <gazebo reference="wheel_3">
+  <!-- <gazebo reference="right_wheel">
     <mu1>10000</mu1>
     <mu2>10000</mu2>
@@ -44,11 +44,11 @@
     <material>Gazebo/Grey</material>
   </gazebo> -->
-  <!-- <gazebo>
+  <gazebo>
     <plugin name="gazebo_ros_control" filename="libgazebo_ros_control.so">
       <robotNamespace>/librarian</robotNamespace>
       <robotSimType>gazebo_ros_control/DefaultRobotHWSim</robotSimType>
     </plugin>
- </gazebo> -->
-  <gazebo>
+ </gazebo>
+  <!-- <gazebo>
     <plugin name="object_controller" filename="libgazebo_ros_planar_move.so">
       <commandTopic>cmd_vel</commandTopic>
@@ -58,5 +58,5 @@
       <robotBaseFrame>base_link</robotBaseFrame>
     </plugin>
-  </gazebo>
+  </gazebo> -->
   <!-- <gazebo reference="imu_link">
     <gravity>true</gravity>
@@ -111,5 +111,5 @@
     <sensor type="ray" name="lds_lfcd_sensor">
       <pose>0 0 0 0 0 0</pose>
-      <visualize>$(arg laser_visual)</visualize>
+      <visualize>false</visualize>
       <update_rate>5</update_rate>
       <ray>

File: lib_omni_mobile/urdf/omni_mobile.urdf.xacro (robot description, xacro)
@@ -1,122 +1,35 @@
 <?xml version="1.0"?>
-<robot xmlns:xacro="http://www.ros.org/wiki/xacro" name="omni_mobile">
-    <xacro:include filename="$(find lib_omni_mobile)/urdf/materials.xacro" />
-	<xacro:include filename="$(find lib_omni_mobile)/urdf/roller_wheel.urdf.xacro"/>
+<robot name="omni_mobile" xmlns:xacro="http://www.ros.org/wiki/xacro">
+	<xacro:include filename="$(find lib_omni_mobile)/urdf/rim_wheel.urdf.xacro"/>
 	<xacro:include filename="$(find lib_omni_mobile)/urdf/omni_mobile.gazebo.xacro" />
 	<xacro:property name="PI" value="3.14" />
-    <xacro:property name="base_link_length" value="0.1" />
+    <xacro:property name="base_link_length" value="0.07" />
     <xacro:property name="base_link_radius" value="0.15" />
-	<xacro:property name="wheel_length" value="0.035" />
-	<xacro:property name="wheel_radius" value="0.1" />
+	<xacro:property name="wheel_length" value="0.04" />
+	<xacro:property name="wheel_radius" value="0.04" />
     <link name="base_link">
 		<visual>
 			<geometry>
 				<cylinder length="${base_link_length}" radius="${base_link_radius}"/>
-				<!-- <mesh filename="package://lib_omni_mobile/meshes/base.STL" scale="0.001 0.001 0.001"/> -->
 			</geometry>
-			<origin xyz="0 0 ${base_link_length/2+wheel_radius/2}"/>
-			<!-- <origin xyz="0 0 0" rpy="1.5708 0 0"/> -->
-			<material name="blue"/>
+			<origin xyz="0 0 ${base_link_length/2+wheel_radius}" rpy="0 0 0"/>
+			<material name="white"/>
 		</visual>
 		<collision>
 			<geometry>
 				<cylinder length="${base_link_length}" radius="${base_link_radius}"/>
-				<!-- <mesh filename="package://lib_omni_mobile/meshes/base.STL" scale="0.001 0.001 0.001"/> -->
 			</geometry>
-			<origin xyz="0 0 ${base_link_length/2+wheel_radius/2}"/>
-			<!-- <origin xyz="0 0 0" rpy="1.5708 0 0"/> -->
-			<material name="blue"/>
-		</collision>
-	</link>
-	<joint name="jwheel_1" type="continuous">
-		<parent link="base_link"/>
-		<child link="wheel_1"/>
-		<origin xyz="${base_link_radius+wheel_length/2} 0 ${base_link_length}" rpy="0 ${PI/2} ${PI/2}"/>
-		<axis xyz="0 0 1"/>
-		<limit effort="1000" lower="${-PI}" upper="${PI}" velocity="5"/>
-	</joint>
-	<link name="wheel_1">
-		<visual>
-			<geometry>
-				<cylinder length="${wheel_length}" radius="${wheel_radius}"/>
-			</geometry>
-			<origin xyz="0 0 0" rpy="1.57 0 0"/>
-			<material name="black"/>
-		</visual>
-		<collision>
-			<geometry>
-				<cylinder length="${wheel_length}" radius="${wheel_radius}"/>
-			</geometry>
-			<origin xyz="0 0 0" rpy="0 0 0"/>
-			<material name="black"/>
+			<origin xyz="0 0 ${base_link_length/2+wheel_radius}" rpy="0 0 0"/>
+			<material name="white"/>
 		</collision>
 		<inertial>
-			<origin xyz="0 0 0" />
-			<mass value="2.8498940e-02" />
-			<inertia ixx="1.1175580e-05" ixy="-4.2369783e-11" ixz="-5.9381719e-09"
-					iyy="1.1192413e-05" iyz="-1.4400107e-11"
-					izz="2.0712558e-05" />
-      	</inertial>
+			<origin xyz="0 0 0" rpy="0 0 0"/>
+			<mass value="0.10"/>
+			<inertia ixx="0.00092" ixy="0.0" ixz="0.0" iyy="0.00178" iyz="0.0" izz="0.00092"/>
+		</inertial>
 	</link>
-	<joint name="jwheel_2" type="continuous">
-		<parent link="base_link"/>
-		<child link="wheel_2"/>
-		<origin xyz="${-0.5*(base_link_radius+wheel_length/2)} ${0.866*(base_link_radius+wheel_length/2)} ${base_link_length}" rpy="0 ${PI/2} ${7*PI/6}"/>
-		<axis xyz="0 0 1"/>
-		<limit effort="1000" lower="${-PI}" upper="${PI}" velocity="5"/>
-	</joint>
-	<link name="wheel_2">
-		<visual>
-			<geometry>
-				<cylinder length="${wheel_length}" radius="${wheel_radius}"/>
-			</geometry>
-			<origin xyz="0 0 0" rpy="1.57 0 0"/>
-			<material name="black"/>
-		</visual>
-		<collision>
-			<geometry>
-				<cylinder length="${wheel_length}" radius="${wheel_radius}"/>
-			</geometry>
-			<origin xyz="0 0 0" rpy="0 0 0"/>
-			<material name="black"/>
-		</collision>
-		<inertial>
-			<origin xyz="0 0 0" />
-			<mass value="2.8498940e-02" />
-			<inertia ixx="1.1175580e-05" ixy="-4.2369783e-11" ixz="-5.9381719e-09"
-					iyy="1.1192413e-05" iyz="-1.4400107e-11"
-					izz="2.0712558e-05" />
-      	</inertial>
-	</link>
-	<joint name="jwheel_3" type="continuous">
-		<parent link="base_link"/>
-		<child link="wheel_3"/>
-		<origin xyz="${-0.5*(base_link_radius+wheel_length/2)} ${-0.866*(base_link_radius+wheel_length/2)} ${base_link_length}" rpy="0 ${PI/2} ${-PI/6}"/>
-		<axis xyz="0 0 1"/>
-		<limit effort="1000" lower="${-PI}" upper="${PI}" velocity="5"/>
-	</joint>
-	<link name="wheel_3">
-		<visual>
-			<geometry>
-				<cylinder length="${wheel_length}" radius="${wheel_radius}"/>
-			</geometry>
-			<origin xyz="0 0 0" rpy="1.57 0 0"/>
-			<material name="black"/>
-		</visual>
-		<collision>
-			<geometry>
-				<cylinder length="${wheel_length}" radius="${wheel_radius}"/>
-			</geometry>
-			<origin xyz="0 0 0" rpy="0 0 0"/>
-			<material name="black"/>
-		</collision>
-		<inertial>
-			<origin xyz="0 0 0" />
-			<mass value="2.8498940e-02" />
-			<inertia ixx="1.1175580e-05" ixy="-4.2369783e-11" ixz="-5.9381719e-09"
-					iyy="1.1192413e-05" iyz="-1.4400107e-11"
-					izz="2.0712558e-05" />
-      	</inertial>
-	</link>
+	<xacro:rim name="left_wheel" parent="base_link" xyz="${-0.5*(base_link_radius+wheel_length/2)} ${0.866*(base_link_radius+wheel_length/2)} ${base_link_length}" rpy="0 ${PI/2} ${2*PI/3}"/>
+	<xacro:rim name="right_wheel" parent="base_link" xyz="${-0.5*(base_link_radius+wheel_length/2)} ${-0.866*(base_link_radius+wheel_length/2)} ${base_link_length}" rpy="0 ${PI/2} ${-2*PI/3}"/>
+	<xacro:rim name="front_wheel" parent="base_link" xyz="${base_link_radius+wheel_length/2} 0 ${base_link_length}" rpy="0 ${PI/2} ${PI}"/>
 	<joint name="scan_joint" type="fixed">
 		<parent link="base_link"/>
@@ -133,18 +46,4 @@
 			<material name="dark"/>
 		</visual>
-		<collision>
-			<geometry>
-				<cylinder length="0.0315" radius="0.045"/>
-			</geometry>
-			<origin xyz="0.015 0 -0.0065"  rpy="0 0 0"/>
-			<material name="dark"/>
-		</collision>
-		<inertial>
-			<mass value="0.114" />
-			<origin xyz="0 0 0" />
-			<inertia ixx="0.001" ixy="0.0" ixz="0.0"
-					iyy="0.001" iyz="0.0"
-					izz="0.001" />
-		</inertial>
 	</link>
 </robot>

File: lib_omni_mobile/urdf/roller_wheel.urdf.xacro (robot description, xacro)
@@ -2,5 +2,5 @@
 <robot xmlns:xacro="http://www.ros.org/wiki/xacro">
 <xacro:macro name="roller" params="name parent xyz rpy">
-    <link name="roller_${name}_rim_${parent}_link">
+    <link name="roller_${name}_${parent}">
         <inertial>
             <inertia ixx="1e-6" ixy="0.0" ixz="0.0" iyy="1e-6" iyz="0.0" izz="1e-7"/>
@@ -9,16 +9,16 @@
         <visual>
             <geometry>
-                <cylinder radius="0.01" length="0.03"/>
+                <cylinder radius="0.01" length="0.02"/>
             </geometry>
         </visual>
         <collision>
             <geometry>
-                <cylinder radius="0.01" length="0.03"/>
+                <cylinder radius="0.01" length="0.02"/>
             </geometry>
         </collision>
     </link>
-    <joint name="roller_${name}_rim_${parent}_joint" type="continuous">
-        <parent link="rim_${parent}_link"/>
-        <child link="roller_${name}_rim_${parent}_link"/>
+    <joint name="roller_${name}_${parent}" type="fixed">
+        <parent link="${parent}"/>
+        <child link="roller_${name}_${parent}"/>
         <axis xyz="0 0 1"/>
         <origin xyz="${xyz}" rpy="${rpy}"/>

File: lib_planar_arm/urdf/planar_arm.urdf.xacro (robot description, xacro)
@@ -1,5 +1,4 @@
 <?xml version="1.0"?>
 <robot xmlns:xacro="http://www.ros.org/wiki/xacro" name="planar_arm">
-    <xacro:include filename="$(find lib_planar_arm)/urdf/materials.xacro" />
 	<xacro:property name="offset" value="0.02" />
     <xacro:property name="base_link_length" value="0.05" />
@@ -9,5 +8,5 @@
 	<xacro:property name="link2_length" value="0.20" />
 	<xacro:property name="link3_length" value="0.20" />
-    <link name="base_link">
+    <link name="planar_link">
 		<visual>
 			<geometry>
@@ -26,5 +25,5 @@
 	</link>
 	<joint name="joint_1" type="revolute">
-		<parent link="base_link"/>
+		<parent link="planar_link"/>
 		<child link="link_1"/>
 		<origin xyz="0.0 ${link_width} ${base_link_length+offset}"/>

Commit message: Update Omni

File: lib_bringup/urdf/librarian.urdf.xacro (robot description, xacro)
@@ -5,10 +5,10 @@
   <xacro:include filename="$(find lib_omni_mobile)/urdf/omni_mobile.urdf.xacro" />
   <!-- Include Planar Arm URDF -->
-  <xacro:include filename="$(find lib_planar_arm)/urdf/planar_arm.urdf.xacro" />
+  <!-- <xacro:include filename="$(find lib_planar_arm)/urdf/planar_arm.urdf.xacro" /> -->
   <!-- Base fixed joint -->
-  <joint name="base_fixed" type="fixed">
+  <!-- <joint name="base_fixed" type="fixed">
     <origin xyz="0.0 0.0 0.0" rpy="0 0 0"/>
     <parent link="base_link"/>
     <child link="planar_link"/>
-  </joint>
+  </joint> -->
 </robot>

File: lib_omni_mobile/urdf/omni_mobile.gazebo.xacro (robot description, xacro)
@@ -84,5 +84,5 @@
       <bodyName>imu_link</bodyName>
       <frameName>imu_link</frameName>
-      <topicName>omni_mobile/imu_data</topicName>
+      <topicName>librarian/imu_data</topicName>
       <serviceName>imu_service</serviceName>
       <gaussianNoise>0.0</gaussianNoise>

File: lib_omni_mobile/urdf/omni_mobile.urdf.xacro (robot description, xacro)
@@ -47,3 +47,9 @@
 		</visual>
 	</link>
+	<!-- <joint name="imu_joint" type="fixed">
+    	<parent link="base_link"/>
+    	<child link="imu_link"/>
+    	<origin xyz="0.0 0.0 0.0" rpy="0 0 0"/>
+  	</joint>
+  	<link name="imu_link"/> -->
 </robot>

File: lib_omni_mobile/urdf/roller_wheel.urdf.xacro (robot description, xacro)
@@ -18,5 +18,5 @@
         </collision>
     </link>
-    <joint name="roller_${name}_${parent}" type="fixed">
+    <joint name="roller_${name}_${parent}" type="continuous">
         <parent link="${parent}"/>
         <child link="roller_${name}_${parent}"/>

Commit message: Update code

File: lib_bringup/urdf/librarian.urdf.xacro (robot description, xacro)
@@ -5,10 +5,10 @@
   <xacro:include filename="$(find lib_omni_mobile)/urdf/omni_mobile.urdf.xacro" />
   <!-- Include Planar Arm URDF -->
-  <!-- <xacro:include filename="$(find lib_planar_arm)/urdf/planar_arm.urdf.xacro" /> -->
+  <xacro:include filename="$(find lib_planar_arm)/urdf/planar_arm.urdf.xacro" />
   <!-- Base fixed joint -->
-  <!-- <joint name="base_fixed" type="fixed">
+  <joint name="base_fixed" type="fixed">
     <origin xyz="0.0 0.0 0.0" rpy="0 0 0"/>
     <parent link="base_link"/>
     <child link="planar_link"/>
-  </joint> -->
+  </joint>
 </robot>

File: lib_omni_mobile/urdf/omni_mobile.urdf.xacro (robot description, xacro)
@@ -43,5 +43,6 @@
 			<origin xyz="0 0 0"/>
 			<geometry>
-				<mesh filename="package://turtlebot3_description/meshes/sensors/lds.stl" scale="0.001 0.001 0.001"/>
+				<!-- <mesh filename="package://turtlebot3_description/meshes/sensors/lds.stl" scale="0.001 0.001 0.001"/> -->
+				<cylinder length="0.05" radius="0.02"/>
 			</geometry>
 			<origin xyz="0 0 0" rpy="0 0 0"/>
